File: KiCad/pressure_sensor.kicad_sch (KiCad schematic)
At the start: 9 parts, among them IC3 MS5849-30BA, U14 SN74LV1T34DCK, U7 SN74LV1T34DCK, U8 PCA9306

Commit message: Create Revision 0.0.1
Other:
- company: (none) -> ETH Zurich: Center for Project Based Learning
- title: (none) -> STDC: Pressure Sensor
Changed lines of the file:
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@@
 	(generator_version "9.0")
 	(paper "A4")
+	(title_block
+		(title "STDC: Pressure Sensor")
+		(date "2026-03-05")
+		(rev "0.0.1")
+		(company "ETH Zurich: Center for Project Based Learning")
+	)
 	(rectangle
 		(start 58.42 45.72)

Commit message: Added some TODOs, fixed some TODOs
Parts:
- added C53, C54, C56: 100n, Capacitor_SMD:C_0402_1005Metric, symbol Device:C
- renumbered C49 to C55
Connections:
- net +1V8: now also C53.1, C56.1
- net +3.3V: now also C54.1
- net GND: now also C53.2, C54.2, C56.2
Other:
- moved on the sheet: C55, IC3, U7

Commit message: Testing connectors, SPI2 pinout, reannotate
Parts:
- renumbered R25 to R26, R26 to R27, R27 to R28, R28 to R29, U14 to U7, U7 to U8, U8 to U9
Changed lines of the file:
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@@
 	(wire
 		(pts
-			(xy 132.08 60.96) (xy 123.19 60.96)
+			(xy 128.27 60.96) (xy 123.19 60.96)
 		)
 		(stroke
@@
 	(wire
 		(pts
-			(xy 105.41 82.55) (xy 132.08 82.55)
+			(xy 105.41 82.55) (xy 128.27 82.55)
 		)
 		(stroke
@@
 	(wire
 		(pts
-			(xy 132.08 60.96) (xy 132.08 82.55)
+			(xy 128.27 60.96) (xy 128.27 82.55)
 		)
 		(stroke
@@
 	)
 	(label "Pressure_EN_3V3"
-		(at 132.08 81.28 90)
+		(at 128.27 81.28 90)
 		(effects
 			(font
@@
 		(on_board yes)
 		(dnp no)
-		(property "Reference" "R27"
+		(property "Reference" "R28"
 			(at 77.47 67.31 0)
 			(effects
@@
 			(project "STDC"
 				(path "/643c756f-a801-466b-9148-7370ee6a5e00/6d95f2ec-8262-4bee-9f8d-5095f2202482"
-					(reference "R27")
+					(reference "R28")
 					(unit 1)
 				)
@@
 		(on_board yes)
 		(dnp no)
-		(property "Reference" "#PWR036"
+		(property "Reference" "#PWR034"
 			(at 195.58 54.61 0)
 			(effects
@@
 			(project ""
 				(path "/643c756f-a801-466b-9148-7370ee6a5e00/6d95f2ec-8262-4bee-9f8d-5095f2202482"
-					(reference "#PWR036")
+					(reference "#PWR034")
 					(unit 1)
 				)
@@
 		(on_board yes)
 		(dnp no)
-		(property "Reference" "R25"
+		(property "Reference" "R26"
 			(at 137.16 66.04 0)
 			(effects
@@
 			(project "STDC"
 				(path "/643c756f-a801-466b-9148-7370ee6a5e00/6d95f2ec-8262-4bee-9f8d-5095f2202482"
-					(reference "R25")
+					(reference "R26")
 					(unit 1)
 				)
@@
 		(on_board yes)
 		(dnp no)
-		(property "Reference" "#PWR038"
+		(property "Reference" "#PWR037"
 			(at 95.25 107.95 0)
 			(effects
@@
 			(project "STDC"
 				(path "/643c756f-a801-466b-9148-7370ee6a5e00/6d95f2ec-8262-4bee-9f8d-5095f2202482"
-					(reference "#PWR038")
+					(reference "#PWR037")
 					(unit 1)
 				)
@@
 		(on_board yes)
 		(dnp no)
-		(property "Reference" "#PWR035"
+		(property "Reference" "#PWR033"
 			(at 147.32 54.61 0)
 			(effects
@@
 			(project "STDC"
 				(path "/643c756f-a801-466b-9148-7370ee6a5e00/6d95f2ec-8262-4bee-9f8d-5095f2202482"
-					(reference "#PWR035")
+					(reference "#PWR033")
 					(unit 1)
 				)
@@
 		(on_board yes)
 		(dnp no)
-		(property "Reference" "#PWR037"
+		(property "Reference" "#PWR035"
 			(at 222.25 54.61 0)
 			(effects
@@
 			(project "STDC"
 				(path "/643c756f-a801-466b-9148-7370ee6a5e00/6d95f2ec-8262-4bee-9f8d-5095f2202482"
-					(reference "#PWR037")
+					(reference "#PWR035")
 					(unit 1)
 				)
@@
 		(on_board yes)
 		(dnp no)
-		(property "Reference" "U14"
+		(property "Reference" "U7"
 			(at 111.506 54.61 0)
 			(effects
@@
 			(project "STDC"
 				(path "/643c756f-a801-466b-9148-7370ee6a5e00/6d95f2ec-8262-4bee-9f8d-5095f2202482"
-					(reference "U14")
+					(reference "U7")
 					(unit 1)
 				)
@@
 		(on_board yes)
 		(dnp no)
-		(property "Reference" "#PWR039"
+		(property "Reference" "#PWR036"
 			(at 146.05 106.68 0)
 			(effects
@@
 			(project ""
 				(path "/643c756f-a801-466b-9148-7370ee6a5e00/6d95f2ec-8262-4bee-9f8d-5095f2202482"
-					(reference "#PWR039")
+					(reference "#PWR036")
 					(unit 1)
 				)
@@
 		(on_board yes)
 		(dnp no)
-		(property "Reference" "U7"
+		(property "Reference" "U8"
 			(at 218.186 73.66 0)
 			(effects
@@
 			(project ""
 				(path "/643c756f-a801-466b-9148-7370ee6a5e00/6d95f2ec-8262-4bee-9f8d-5095f2202482"
-					(reference "U7")
+					(reference "U8")
 					(unit 1)
 				)
@@
 		(on_board yes)
 		(dnp no)
-		(property "Reference" "U8"
+		(property "Reference" "U9"
 			(at 88.9 96.52 0)
 			(effects
@@
 			(project ""
 				(path "/643c756f-a801-466b-9148-7370ee6a5e00/6d95f2ec-8262-4bee-9f8d-5095f2202482"
-					(reference "U8")
+					(reference "U9")
 					(unit 1)
 				)
@@
 		(on_board yes)
 		(dnp no)
-		(property "Reference" "R28"
+		(property "Reference" "R29"
 			(at 83.82 67.31 0)
 			(effects
@@
 			(project "STDC"
 				(path "/643c756f-a801-466b-9148-7370ee6a5e00/6d95f2ec-8262-4bee-9f8d-5095f2202482"
-					(reference "R28")
+					(reference "R29")
 					(unit 1)
 				)
@@
 		(on_board yes)
 		(dnp no)
-		(property "Reference" "R26"
+		(property "Reference" "R27"
 			(at 143.51 66.04 0)
 			(effects
@@
 			(project ""
 				(path "/643c756f-a801-466b-9148-7370ee6a5e00/6d95f2ec-8262-4bee-9f8d-5095f2202482"
-					(reference "R26")
+					(reference "R27")
 					(unit 1)
 				)
@@
 		(on_board yes)
 		(dnp no)
-		(property "Reference" "#PWR034"
+		(property "Reference" "#PWR032"
 			(at 92.71 54.61 0)
 			(effects
@@
 			(project ""
 				(path "/643c756f-a801-466b-9148-7370ee6a5e00/6d95f2ec-8262-4bee-9f8d-5095f2202482"
-					(reference "#PWR034")
+					(reference "#PWR032")
 					(unit 1)
 				)

Commit message: Calculate saturation current for coils and add comments
Parts:
- renumbered C53 to C55, C54 to C56, C55 to C57, C56 to C58
Changed lines of the file:
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@@
 		(on_board yes)
 		(dnp no)
-		(property "Reference" "C55"
+		(property "Reference" "C57"
 			(at 162.56 73.66 0)
 			(effects
@@
 			(project "STDC"
 				(path "/643c756f-a801-466b-9148-7370ee6a5e00/6d95f2ec-8262-4bee-9f8d-5095f2202482"
-					(reference "C55")
+					(reference "C57")
 					(unit 1)
 				)
@@
 		(on_board yes)
 		(dnp no)
-		(property "Reference" "C53"
+		(property "Reference" "C55"
 			(at 69.85 71.12 0)
 			(effects
@@
 			(project "STDC"
 				(path "/643c756f-a801-466b-9148-7370ee6a5e00/6d95f2ec-8262-4bee-9f8d-5095f2202482"
-					(reference "C53")
+					(reference "C55")
 					(unit 1)
 				)
@@
 		(on_board yes)
 		(dnp no)
-		(property "Reference" "C56"
+		(property "Reference" "C58"
 			(at 242.57 90.17 0)
 			(effects
@@
 			(project "STDC"
 				(path "/643c756f-a801-466b-9148-7370ee6a5e00/6d95f2ec-8262-4bee-9f8d-5095f2202482"
-					(reference "C56")
+					(reference "C58")
 					(unit 1)
 				)
@@
 		(on_board yes)
 		(dnp no)
-		(property "Reference" "C54"
+		(property "Reference" "C56"
 			(at 152.4 73.66 0)
 			(effects
@@
 			(project "STDC"
 				(path "/643c756f-a801-466b-9148-7370ee6a5e00/6d95f2ec-8262-4bee-9f8d-5095f2202482"
-					(reference "C54")
-					(unit 1)
-				)
+					(reference "C56")
+					(unit 1)
+				)

Commit message: First Draft PCB Layout
Parts:
- added C51: 100n, Capacitor_SMD:C_0402_1005Metric, symbol Device:C
- renumbered C55 to C52, C56 to C53, C57 to C54, C58 to C55
Connections:
- net +3.3V: now also C51.1
- net GND: now also C51.2
Changed lines of the file:
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@@
+	)
+	(junction
+		(at 106.68 52.07)
+		(diameter 0)
+		(color 0 0 0 0)
 	)
 	(junction
@@
 	)
 	(junction
+		(at 106.68 99.06)
+		(diameter 0)
+		(color 0 0 0 0)
+	)
+	(junction
 		(at 95.25 99.06)
 		(diameter 0)
@@
 	(wire
 		(pts
+			(xy 106.68 99.06) (xy 95.25 99.06)
+		)
+		(stroke
+			(width 0)
+			(type default)
+		)
+	)
+	(wire
+		(pts
 			(xy 82.55 52.07) (xy 82.55 64.77)
 		)
@@
 	(wire
 		(pts
-			(xy 115.57 99.06) (xy 95.25 99.06)
+			(xy 115.57 99.06) (xy 106.68 99.06)
 		)
 		(stroke
@@
 	(wire
 		(pts
+			(xy 106.68 66.04) (xy 106.68 52.07)
+		)
+		(stroke
+			(width 0)
+			(type default)
+		)
+	)
+	(wire
+		(pts
 			(xy 142.24 52.07) (xy 147.32 52.07)
 		)
@@
 	(wire
 		(pts
+			(xy 106.68 73.66) (xy 106.68 99.06)
+		)
+		(stroke
+			(width 0)
+			(type default)
+		)
+	)
+	(wire
+		(pts
 			(xy 142.24 71.12) (xy 142.24 87.63)
 		)
@@
 	(wire
 		(pts
+			(xy 106.68 52.07) (xy 115.57 52.07)
+		)
+		(stroke
+			(width 0)
+			(type default)
+		)
+	)
+	(wire
+		(pts
 			(xy 149.86 69.85) (xy 160.02 69.85)
 		)
@@
 	(wire
 		(pts
-			(xy 97.79 52.07) (xy 115.57 52.07)
+			(xy 97.79 52.07) (xy 106.68 52.07)
 		)
 		(stroke
@@
 		(on_board yes)
 		(dnp no)
-		(property "Reference" "C57"
+		(property "Reference" "C54"
 			(at 162.56 73.66 0)
 			(effects
@@
 			(project "STDC"
 				(path "/643c756f-a801-466b-9148-7370ee6a5e00/6d95f2ec-8262-4bee-9f8d-5095f2202482"
-					(reference "C57")
+					(reference "C54")
 					(unit 1)
 				)
@@
 		(on_board yes)
 		(dnp no)
-		(property "Reference" "#PWR034"
+		(property "Reference" "#PWR031"
 			(at 195.58 54.61 0)
 			(effects
@@
 			(project ""
 				(path "/643c756f-a801-466b-9148-7370ee6a5e00/6d95f2ec-8262-4bee-9f8d-5095f2202482"
-					(reference "#PWR034")
+					(reference "#PWR031")
 					(unit 1)
 				)
@@
 		(on_board yes)
 		(dnp no)
-		(property "Reference" "C55"
+		(property "Reference" "C52"
 			(at 69.85 71.12 0)
 			(effects
@@
 			(project "STDC"
 				(path "/643c756f-a801-466b-9148-7370ee6a5e00/6d95f2ec-8262-4bee-9f8d-5095f2202482"
-					(reference "C55")
+					(reference "C52")
 					(unit 1)
 				)
@@
 		(on_board yes)
 		(dnp no)
-		(property "Reference" "C58"
+		(property "Reference" "C55"
 			(at 242.57 90.17 0)
 			(effects
@@
 			(project "STDC"
 				(path "/643c756f-a801-466b-9148-7370ee6a5e00/6d95f2ec-8262-4bee-9f8d-5095f2202482"
-					(reference "C58")
+					(reference "C55")
 					(unit 1)
 				)
@@
 		(on_board yes)
 		(dnp no)
-		(property "Reference" "C56"
+		(property "Reference" "C53"
 			(at 152.4 73.66 0)
 			(effects
@@
 			(project "STDC"
 				(path "/643c756f-a801-466b-9148-7370ee6a5e00/6d95f2ec-8262-4bee-9f8d-5095f2202482"
-					(reference "C56")
+					(reference "C53")
 					(unit 1)
 				)
@@
 		(on_board yes)
 		(dnp no)
-		(property "Reference" "#PWR037"
+		(property "Reference" "#PWR034"
 			(at 95.25 107.95 0)
 			(effects
@@
 			(project "STDC"
 				(path "/643c756f-a801-466b-9148-7370ee6a5e00/6d95f2ec-8262-4bee-9f8d-5095f2202482"
-					(reference "#PWR037")
+					(reference "#PWR034")
 					(unit 1)
 				)
@@
 		(on_board yes)
 		(dnp no)
-		(property "Reference" "#PWR033"
+		(property "Reference" "#PWR030"
 			(at 147.32 54.61 0)
 			(effects
@@
 			(project "STDC"
 				(path "/643c756f-a801-466b-9148-7370ee6a5e00/6d95f2ec-8262-4bee-9f8d-5095f2202482"
-					(reference "#PWR033")
+					(reference "#PWR030")
 					(unit 1)
 				)
@@
 		(on_board yes)
 		(dnp no)
-		(property "Reference" "#PWR035"
+		(property "Reference" "#PWR032"
 			(at 222.25 54.61 0)
 			(effects
@@
 			(project "STDC"
 				(path "/643c756f-a801-466b-9148-7370ee6a5e00/6d95f2ec-8262-4bee-9f8d-5095f2202482"
-					(reference "#PWR035")
+					(reference "#PWR032")
 					(unit 1)
 				)
@@
 	)
 	(symbol
+		(lib_id "Device:C")
+		(at 106.68 69.85 0)
+		(unit 1)
+		(exclude_from_sim no)
+		(in_bom yes)
+		(on_board yes)
+		(dnp no)
+		(property "Reference" "C51"
+			(at 109.22 68.58 0)
+			(effects
+				(font
+					(size 1.27 1.27)
+				)
+				(justify left)
+			)
+		)
+		(property "Value" "100n"
+			(at 109.22 71.12 0)
+			(effects
+				(font
+					(size 1.27 1.27)
+				)
+				(justify left)
+			)
+		)
+		(property "Footprint" "Capacitor_SMD:C_0402_1005Metric"
+			(at 107.6452 73.66 0)
+			(effects
+				(font
+					(size 1.27 1.27)
+				)
+				(hide yes)
+			)
+		)
+		(property "Datasheet" "~"
+			(at 106.68 69.85 0)
+			(effects
+				(font
+					(size 1.27 1.27)
+				)
+				(hide yes)
+			)
+		)
+		(property "Description" "Unpolarized capacitor"
+			(at 106.68 69.85 0)
+			(effects
+				(font
+					(size 1.27 1.27)
+				)
+				(hide yes)
+			)
+		)
+		(pin "2"
+		)
+		(pin "1"
+		)
+		(instances
+			(project "STDC"
+				(path "/643c756f-a801-466b-9148-7370ee6a5e00/6d95f2ec-8262-4bee-9f8d-5095f2202482"
+					(reference "C51")
+					(unit 1)
+				)
+			)
+		)
+	)
+	(symbol
 		(lib_id "power:GND")
 		(at 146.05 100.33 0)
@@
 		(on_board yes)
 		(dnp no)
-		(property "Reference" "#PWR036"
+		(property "Reference" "#PWR033"
 			(at 146.05 106.68 0)
 			(effects
@@
 			(project ""
 				(path "/643c756f-a801-466b-9148-7370ee6a5e00/6d95f2ec-8262-4bee-9f8d-5095f2202482"
-					(reference "#PWR036")
+					(reference "#PWR033")
 					(unit 1)
 				)
@@
 		(on_board yes)
 		(dnp no)
-		(property "Reference" "#PWR032"
+		(property "Reference" "#PWR029"
 			(at 92.71 54.61 0)
 			(effects
@@
 			(project ""
 				(path "/643c756f-a801-466b-9148-7370ee6a5e00/6d95f2ec-8262-4bee-9f8d-5095f2202482"
-					(reference "#PWR032")
+					(reference "#PWR029")
 					(unit 1)
 				)

Commit message: Implement Comments, Working on PCB Layout
Parts:
- renumbered C51 to C48, C52 to C49, C53 to C50, C54 to C51, C55 to C52, IC3 to IC4, R26 to R20, R27 to R21, R28 to R22, R29 to R23
Changed lines of the file:
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@@
 		(on_board yes)
 		(dnp no)
-		(property "Reference" "R28"
+		(property "Reference" "R22"
 			(at 77.47 67.31 0)
 			(effects
@@
 			(project "STDC"
 				(path "/643c756f-a801-466b-9148-7370ee6a5e00/6d95f2ec-8262-4bee-9f8d-5095f2202482"
-					(reference "R28")
+					(reference "R22")
 					(unit 1)
 				)
@@
 		(on_board yes)
 		(dnp no)
-		(property "Reference" "C54"
+		(property "Reference" "C51"
 			(at 162.56 73.66 0)
 			(effects
@@
 			(project "STDC"
 				(path "/643c756f-a801-466b-9148-7370ee6a5e00/6d95f2ec-8262-4bee-9f8d-5095f2202482"
-					(reference "C54")
+					(reference "C51")
 					(unit 1)
 				)
@@
 		(on_board yes)
 		(dnp no)
-		(property "Reference" "C52"
+		(property "Reference" "C49"
 			(at 69.85 71.12 0)
 			(effects
@@
 			(project "STDC"
 				(path "/643c756f-a801-466b-9148-7370ee6a5e00/6d95f2ec-8262-4bee-9f8d-5095f2202482"
-					(reference "C52")
+					(reference "C49")
 					(unit 1)
 				)
@@
 		(on_board yes)
 		(dnp no)
-		(property "Reference" "C55"
+		(property "Reference" "C52"
 			(at 242.57 90.17 0)
 			(effects
@@
 			(project "STDC"
 				(path "/643c756f-a801-466b-9148-7370ee6a5e00/6d95f2ec-8262-4bee-9f8d-5095f2202482"
-					(reference "C55")
+					(reference "C52")
 					(unit 1)
 				)
@@
 		(on_board yes)
 		(dnp no)
-		(property "Reference" "C53"
+		(property "Reference" "C50"
 			(at 152.4 73.66 0)
 			(effects
@@
 			(project "STDC"
 				(path "/643c756f-a801-466b-9148-7370ee6a5e00/6d95f2ec-8262-4bee-9f8d-5095f2202482"
-					(reference "C53")
+					(reference "C50")
 					(unit 1)
 				)
@@
 		(on_board yes)
 		(dnp no)
-		(property "Reference" "R26"
+		(property "Reference" "R20"
 			(at 137.16 66.04 0)
 			(effects
@@
 			(project "STDC"
 				(path "/643c756f-a801-466b-9148-7370ee6a5e00/6d95f2ec-8262-4bee-9f8d-5095f2202482"
-					(reference "R26")
+					(reference "R20")
 					(unit 1)
 				)
@@
 		(on_board yes)
 		(dnp no)
-		(property "Reference" "C51"
+		(property "Reference" "C48"
 			(at 109.22 68.58 0)
 			(effects
@@
 			(project "STDC"
 				(path "/643c756f-a801-466b-9148-7370ee6a5e00/6d95f2ec-8262-4bee-9f8d-5095f2202482"
-					(reference "C51")
+					(reference "C48")
 					(unit 1)
 				)
@@
 		(dnp no)
 		(fields_autoplaced yes)
-		(property "Reference" "IC3"
+		(property "Reference" "IC4"
 			(at 181.61 72.39 0)
 			(effects
@@
 			(project ""
 				(path "/643c756f-a801-466b-9148-7370ee6a5e00/6d95f2ec-8262-4bee-9f8d-5095f2202482"
-					(reference "IC3")
+					(reference "IC4")
 					(unit 1)
 				)
@@
 		(on_board yes)
 		(dnp no)
-		(property "Reference" "R29"
+		(property "Reference" "R23"
 			(at 83.82 67.31 0)
 			(effects
@@
 			(project "STDC"
 				(path "/643c756f-a801-466b-9148-7370ee6a5e00/6d95f2ec-8262-4bee-9f8d-5095f2202482"
-					(reference "R29")
+					(reference "R23")
 					(unit 1)
 				)
@@
 		(on_board yes)
 		(dnp no)
-		(property "Reference" "R27"
+		(property "Reference" "R21"
 			(at 143.51 66.04 0)
 			(effects
@@
 			(project ""
 				(path "/643c756f-a801-466b-9148-7370ee6a5e00/6d95f2ec-8262-4bee-9f8d-5095f2202482"
-					(reference "R27")
-					(unit 1)
-				)
+					(reference "R21")
+					(unit 1)
+				)

Commit message: PCB Layout V0.1 with errors
Other:
- company: ETH Zurich: Center for Project Based Learning -> ETH Zürich: Center for Project Based Learning
Changed lines of the file:
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@@
 		(date "2026-03-09")
 		(rev "0.0.2")
-		(company "ETH Zurich: Center for Project Based Learning")
+		(company "ETH Zürich: Center for Project Based Learning")
 	)
 	(rectangle
