File: KiCad/STDC.kicad_pcb (KiCad board)
At the start: 4 copper layers, 38 x 48 mm, 126 parts, among them IC1 TPS22916CNYFPR, IC2 TPS22916CNYFPR, IC3 R1200N001A-TR-FE, IC4 MS5849-30BA, IC5 W25Q32JWSNIQ, J1 TC2030, J2 Conn_01x03_BATT, J3 Conn_01x34_NHD_18, Q1 AO3400A, Q2 AO3400A, U1 STM32L476RGTx, U10 SN74LV1T34DCK, U11 SN74LV1T34DCK, U12 RN4871, U13 LM810, U14 SN74LV1T34DCK, U2 DW01A, U3 MAX17262REWL_T, U4 BQ51050BRHL, U5 PAM2306AYPKE, U6 MCP1700x-250xxTT, U7 SN74LV1T34DCK, U8 SN74LV1T34DCK, U9 PCA9306, X1 Q13FC1350000400

Commit message: Power Regulator Layout Adjustment
Parts:
- moved C2 0.46 mm to (137.1, 114.1), turned to 90 degrees
- moved C1 0.44 mm to (138.1, 114.1), turned to 90 degrees
Routing:
- net +1V8: track 150.3 -> 151.0 mm
Changed lines of the file:
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@@
 	(footprint "Capacitor_SMD:C_0402_1005Metric"
 		(layer "F.Cu")
-		(at 137.45 114.35 -90)
+		(at 137.08 114.08 90)
 		(descr "Capacitor SMD 0402 (1005 Metric), square (rectangular) end terminal, IPC-7351 nominal, (Body size source: IPC-SM-782 page 76, https://www.pcb-3d.com/wordpress/wp-content/uploads/ipc-sm-782a_amendment_1_and_2.pdf), generated with kicad-footprint-generator")
 		(tags "capacitor")
 		(property "Reference" "C2"
-			(at 1.85 0.625 90)
+			(at -1.73 -0.3 90)
 			(layer "F.SilkS")
 			(effects
@@
 		(attr smd)
 		(fp_line
-			(start -0.107836 0.36)
-			(end 0.107836 0.36)
+			(start -0.107836 -0.36)
+			(end 0.107836 -0.36)
 			(stroke
 				(width 0.12)
@@
 		)
 		(fp_line
-			(start -0.107836 -0.36)
-			(end 0.107836 -0.36)
+			(start -0.107836 0.36)
+			(end 0.107836 0.36)
 			(stroke
 				(width 0.12)
@@
 		)
 		(pad "1" smd roundrect
-			(at -0.48 0 270)
+			(at -0.48 0 90)
 			(size 0.56 0.62)
 			(layers "F.Cu" "F.Mask" "F.Paste")
@@
 		)
 		(pad "2" smd roundrect
-			(at 0.48 0 270)
+			(at 0.48 0 90)
 			(size 0.56 0.62)
 			(layers "F.Cu" "F.Mask" "F.Paste")
@@
 	(footprint "Capacitor_SMD:C_0402_1005Metric"
 		(layer "F.Cu")
-		(at 138.45 114.35 -90)
+		(at 138.1 114.08 90)
 		(descr "Capacitor SMD 0402 (1005 Metric), square (rectangular) end terminal, IPC-7351 nominal, (Body size source: IPC-SM-782 page 76, https://www.pcb-3d.com/wordpress/wp-content/uploads/ipc-sm-782a_amendment_1_and_2.pdf), generated with kicad-footprint-generator")
 		(tags "capacitor")
 		(property "Reference" "C1"
-			(at 1.85 0.15 270)
+			(at -1.62 0.03 90)
 			(layer "F.SilkS")
 			(effects
@@
 		(attr smd)
 		(fp_line
-			(start -0.107836 0.36)
-			(end 0.107836 0.36)
+			(start -0.107836 -0.36)
+			(end 0.107836 -0.36)
 			(stroke
 				(width 0.12)
@@
 		)
 		(fp_line
-			(start -0.107836 -0.36)
-			(end 0.107836 -0.36)
+			(start -0.107836 0.36)
+			(end 0.107836 0.36)
 			(stroke
 				(width 0.12)
@@
 		)
 		(pad "1" smd roundrect
-			(at -0.48 0 270)
+			(at -0.48 0 90)
 			(size 0.56 0.62)
 			(layers "F.Cu" "F.Mask" "F.Paste")
@@
 		)
 		(pad "2" smd roundrect
-			(at 0.48 0 270)
+			(at 0.48 0 90)
 			(size 0.56 0.62)
 			(layers "F.Cu" "F.Mask" "F.Paste")
@@
 	)
 	(segment
+		(start 139.610514 113.401)
+		(end 139.649 113.401)
+		(width 0.3)
+		(layer "F.Cu")
+		(net 1)
+	)
+	(segment
 		(start 151.9 131.8)
 		(end 151.85 131.85)
@@
 	)
 	(segment
-		(start 139.5 113.4)
-		(end 139.03 113.87)
-		(width 0.3)
-		(layer "F.Cu")
-		(net 1)
-	)
-	(segment
 		(start 141.25 128.65)
 		(end 141.5 128.9)
@@
 	(segment
 		(start 140.13 113.4)
-		(end 139.5 113.4)
+		(end 139.65 113.4)
 		(width 0.3)
 		(layer "F.Cu")
@@
 	)
 	(segment
+		(start 138.1 114.56)
+		(end 138.451514 114.56)
+		(width 0.3)
+		(layer "F.Cu")
+		(net 1)
+	)
+	(segment
 		(start 151.968737 131.731262)
 		(end 151.9 131.8)
@@
 	)
 	(segment
-		(start 141.25 128.65)
-		(end 141.6 128.3)
+		(start 139.649 113.401)
+		(end 139.65 113.4)
 		(width 0.3)
 		(layer "F.Cu")
@@
 	)
 	(segment
-		(start 139.03 113.87)
-		(end 138.45 113.87)
+		(start 141.25 128.65)
+		(end 141.6 128.3)
 		(width 0.3)
 		(layer "F.Cu")
@@
 	)
 	(segment
+		(start 138.451514 114.56)
+		(end 139.610514 113.401)
+		(width 0.3)
+		(layer "F.Cu")
+		(net 1)
+	)
+	(segment
 		(start 152.575 107.3)
 		(end 152.135412 107.3)
@@
 	)
 	(segment
-		(start 138.45 114.83)
-		(end 138.45 115.5)
-		(width 0.3)
-		(layer "F.Cu")
-		(net 2)
-	)
-	(segment
 		(start 144.7 105.3)
 		(end 143.95 106.05)
@@
 	)
 	(segment
+		(start 137.08 113.6)
+		(end 137.08 113.12)
+		(width 0.3)
+		(layer "F.Cu")
+		(net 2)
+	)
+	(segment
 		(start 132.4 141.12)
 		(end 132.4 140.4)
@@
 	)
 	(segment
+		(start 138.1 113.6)
+		(end 138.1 113.1)
+		(width 0.3)
+		(layer "F.Cu")
+		(net 2)
+	)
+	(segment
 		(start 127.24 131.46)
 		(end 127.23 131.45)
@@
 	)
 	(segment
-		(start 137.45 114.83)
-		(end 137.45 115.45)
-		(width 0.3)
-		(layer "F.Cu")
-		(net 2)
-	)
-	(segment
 		(start 138.4 132.24)
 		(end 137.71 132.24)
@@
 	)
 	(via
-		(at 138.45 115.5)
+		(at 137.08 113.12)
 		(size 0.45)
 		(drill 0.2)
@@
 	)
 	(via
+		(at 138.1 113.1)
+		(size 0.45)
+		(drill 0.2)
+		(layers "F.Cu" "B.Cu")
+		(net 2)
+	)
+	(via
 		(at 149.65 111.9)
 		(size 0.45)
@@
 	)
 	(via
-		(at 137.45 115.45)
-		(size 0.45)
-		(drill 0.2)
-		(layers "F.Cu" "B.Cu")
-		(net 2)
-	)
-	(via
 		(at 141.396176 133.103228)
 		(size 0.45)
@@
 				(xy 145.2 111.3) (xy 143.7 109.9) (xy 142.85 109.9) (xy 142.55 109.65) (xy 142.55 109.05) (xy 141.25 108.05)
 				(xy 136.6 108.05) (xy 135.95 108.75) (xy 135.95 110.2) (xy 136.25 110.55) (xy 138.85 110.55) (xy 139.35 110)
-				(xy 140.1 110) (xy 140.5 109.65) (xy 140.5 109) (xy 140.75 108.75) (xy 141.25 108.75) (xy 141.5 109.05)
-				(xy 141.5 110.55) (xy 142.4 111.3) (xy 143.6 111.35) (xy 144.1 111.75) (xy 144.1 112.35) (xy 143.75 112.65)
+				(xy 140.1 110) (xy 140.5 109.65) (xy 140.5 109.2) (xy 140.75 109) (xy 141.15 109) (xy 141.4 109.3)
+				(xy 141.4 110.6) (xy 142.25 111.3) (xy 143.6 111.35) (xy 144.1 111.75) (xy 144.1 112.35) (xy 143.75 112.65)
 			)
 		)
@@
 		(polygon
 			(pts
-				(xy 140.55 111.5) (xy 140.55 109) (xy 140.75 108.8) (xy 141.2 108.8) (xy 141.4 109.05) (xy 141.4 110.65)
+				(xy 140.55 111.5) (xy 140.5 109.2) (xy 140.75 109) (xy 141.15 109) (xy 141.4 109.3) (xy 141.4 110.65)
 				(xy 142.55 111.6) (xy 142.55 112.9) (xy 142.65 113) (xy 143.65 113) (xy 143.75 113.1) (xy 143.75 113.3)
 				(xy 143.65 113.4) (xy 142.65 113.4) (xy 142.55 113.5) (xy 142.55 116.8) (xy 142.4 116.95) (xy 141.45 116.95)
@@
 		(polygon
 			(pts
-				(xy 140.6 113.1) (xy 140.5 113) (xy 137.05 113) (xy 136.45 113.6) (xy 136.45 118.6) (xy 139.15 121.4)
-				(xy 139.15 122.05) (xy 139.4 122.3) (xy 141.55 122.35) (xy 142 121.9) (xy 142 118.2) (xy 142.15 118.05)
-				(xy 147.15 118.05) (xy 147.65 117.55) (xy 147.65 116.25) (xy 146.9 115.55) (xy 143.8 115.55) (xy 143.6 115.75)
-				(xy 142.9 115.75) (xy 142.55 116.15) (xy 142.55 116.7) (xy 142.35 116.95) (xy 141.75 116.95) (xy 140.6 116.1)
+				(xy 140.65 113.2) (xy 140.55 113.1) (xy 139.45 113.1) (xy 138.45 114.05) (xy 136.55 114.05) (xy 136.35 114.25)
+				(xy 136.35 118.55) (xy 139.15 121.4) (xy 139.15 122.05) (xy 139.4 122.3) (xy 141.55 122.35) (xy 142 121.9)
+				(xy 142 118.2) (xy 142.15 118.05) (xy 147.15 118.05) (xy 147.65 117.55) (xy 147.65 116.25) (xy 146.9 115.55)
+				(xy 143.8 115.55) (xy 143.6 115.75) (xy 142.9 115.75) (xy 142.55 116.15) (xy 142.55 116.7) (xy 142.35 116.95)
+				(xy 141.75 116.95) (xy 140.6 116.1)
 			)
 		)
