File: KiCad/flash.kicad_sch (KiCad schematic)
At the start: 5 parts, among them IC4 W25Q32JWSNIQ

Commit message: Implement Comments, Working on PCB Layout
Parts:
- renumbered C60 to C57, IC4 to IC5, R34 to R28, R35 to R29, R36 to R30
Changed lines of the file:
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@@
 		(on_board yes)
 		(dnp no)
-		(property "Reference" "R35"
+		(property "Reference" "R29"
 			(at 210.82 48.26 0)
 			(effects
@@
 			(project "STDC"
 				(path "/643c756f-a801-466b-9148-7370ee6a5e00/a5768ca1-322e-4c77-bc87-c3070b355a8f"
-					(reference "R35")
+					(reference "R29")
 					(unit 1)
 				)
@@
 		(on_board yes)
 		(dnp no)
-		(property "Reference" "R36"
+		(property "Reference" "R30"
 			(at 205.74 66.04 0)
 			(effects
@@
 			(project "STDC"
 				(path "/643c756f-a801-466b-9148-7370ee6a5e00/a5768ca1-322e-4c77-bc87-c3070b355a8f"
-					(reference "R36")
+					(reference "R30")
 					(unit 1)
 				)
@@
 		(on_board yes)
 		(dnp no)
-		(property "Reference" "R34"
+		(property "Reference" "R28"
 			(at 124.46 46.99 0)
 			(effects
@@
 			(project "STDC"
 				(path "/643c756f-a801-466b-9148-7370ee6a5e00/a5768ca1-322e-4c77-bc87-c3070b355a8f"
-					(reference "R34")
+					(reference "R28")
 					(unit 1)
 				)
@@
 		(on_board yes)
 		(dnp no)
-		(property "Reference" "C60"
+		(property "Reference" "C57"
 			(at 196.85 66.04 0)
 			(effects
@@
 			(project "STDC"
 				(path "/643c756f-a801-466b-9148-7370ee6a5e00/a5768ca1-322e-4c77-bc87-c3070b355a8f"
-					(reference "C60")
+					(reference "C57")
 					(unit 1)
 				)
@@
 		(on_board yes)
 		(dnp no)
-		(property "Reference" "IC4"
+		(property "Reference" "IC5"
 			(at 146.812 50.546 0)
 			(effects
@@
 			(project "STDC"
 				(path "/643c756f-a801-466b-9148-7370ee6a5e00/a5768ca1-322e-4c77-bc87-c3070b355a8f"
-					(reference "IC4")
+					(reference "IC5")
 					(unit 1)
 				)

Commit message: PCB Layout V0.1 with errors
Other:
- company: ETH Zurich: Center for Project Based Learning -> ETH Zürich: Center for Project Based Learning
Changed lines of the file:
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@@
 		(date "2026-03-09")
 		(rev "0.0.2")
-		(company "ETH Zurich: Center for Project Based Learning")
+		(company "ETH Zürich: Center for Project Based Learning")
 	)
 	(rectangle
